Commit message: Updated joint limit and ur_driver to python3

File: ur_description/urdf/ur5.urdf.xacro (robot description, xacro)
@@ -101,5 +101,5 @@
       <axis xyz="0 0 1" />
       <xacro:unless value="${joint_limited}">
-        <limit lower="${-2.0 * pi}" upper="${2.0 * pi}" effort="150.0" velocity="3.15"/>
+        <limit lower="-4.2" upper="2.8" effort="150.0" velocity="3.15"/>
         <xacro:if value="${safety_limits}">
           <safety_controller soft_lower_limit="${-2.0 * pi + safety_pos_margin}" soft_upper_limit="${2.0 * pi - safety_pos_margin}" k_position="${safety_k_position}" k_velocity="0.0"/>
@@ -138,5 +138,5 @@
       <axis xyz="0 1 0" />
       <xacro:unless value="${joint_limited}">
-        <limit lower="${-2.0 * pi}" upper="${2.0 * pi}" effort="150.0" velocity="3.15"/>
+        <limit lower="-3.1" upper="-0.4" effort="150.0" velocity="3.15"/>
         <xacro:if value="${safety_limits}">
           <safety_controller soft_lower_limit="${-2.0 * pi + safety_pos_margin}" soft_upper_limit="${2.0 * pi - safety_pos_margin}" k_position="${safety_k_position}" k_velocity="0.0"/>
@@ -175,5 +175,5 @@
       <axis xyz="0 1 0" />
       <xacro:unless value="${joint_limited}">
-        <limit lower="${-pi}" upper="${pi}" effort="150.0" velocity="3.15"/>
+        <limit lower="0.6" upper="2.75" effort="150.0" velocity="3.15"/>
         <xacro:if value="${safety_limits}">
           <safety_controller soft_lower_limit="${-2.0 * pi + safety_pos_margin}" soft_upper_limit="${2.0 * pi - safety_pos_margin}" k_position="${safety_k_position}" k_velocity="0.0"/>
@@ -212,5 +212,5 @@
       <axis xyz="0 1 0" />
       <xacro:unless value="${joint_limited}">
-        <limit lower="${-2.0 * pi}" upper="${2.0 * pi}" effort="28.0" velocity="3.2"/>
+        <limit lower="-1.4" upper="1.1" effort="28.0" velocity="3.2"/>
         <xacro:if value="${safety_limits}">
           <safety_controller soft_lower_limit="${-2.0 * pi + safety_pos_margin}" soft_upper_limit="${2.0 * pi - safety_pos_margin}" k_position="${safety_k_position}" k_velocity="0.0"/>
@@ -249,5 +249,5 @@
       <axis xyz="0 0 1" />
       <xacro:unless value="${joint_limited}">
-        <limit lower="${-2.0 * pi}" upper="${2.0 * pi}" effort="28.0" velocity="3.2"/>
+        <limit lower="-1.7" upper="3.0" effort="28.0" velocity="3.2"/>
         <xacro:if value="${safety_limits}">
           <safety_controller soft_lower_limit="${-2.0 * pi + safety_pos_margin}" soft_upper_limit="${2.0 * pi - safety_pos_margin}" k_position="${safety_k_position}" k_velocity="0.0"/>
@@ -286,5 +286,5 @@
       <axis xyz="0 1 0" />
       <xacro:unless value="${joint_limited}">
-        <limit lower="${-2.0 * pi}" upper="${2.0 * pi}" effort="28.0" velocity="3.2"/>
+        <limit lower="-0.35" upper="4.8" effort="28.0" velocity="3.2"/>
         <xacro:if value="${safety_limits}">
           <safety_controller soft_lower_limit="${-2.0 * pi + safety_pos_margin}" soft_upper_limit="${2.0 * pi - safety_pos_margin}" k_position="${safety_k_position}" k_velocity="0.0"/>

File: ur_description/urdf/ur5_with_eof.urdf (robot description, URDF)
Before this commit: robot ur5_with_eof, 13 links, 12 joints
Joints:
- joint ee_fixed_joint: origin xyz=0.0 0.0823 0.0 rpy=0.0 0.0 1.57079632679 -> xyz=0.0 0.0823 0.0 rpy=0.0 0.0 1.5707963267948966
- joint elbow_joint: limit lower=-3.14159265359 upper=3.14159265359 effort=150.0 velocity=3.15 -> lower=-0.3 upper=2.84 effort=150.0 velocity=3.15
- joint eof_joint: origin xyz=0 0 0.05 rpy=0 0 1.57 -> xyz=0 0 0.05 rpy=0 0 -1.57
- joint shoulder_lift_joint: limit lower=-6.28318530718 upper=6.28318530718 effort=150.0 velocity=3.15 -> lower=-2.1 upper=0.0 effort=150.0 velocity=3.15; origin xyz=0.0 0.13585 0.0 rpy=0.0 1.57079632679 0.0 -> xyz=0.0 0.13585 0.0 rpy=0.0 1.5707963267948966 0.0
- joint shoulder_pan_joint: limit lower=-6.28318530718 upper=6.28318530718 effort=150.0 velocity=3.15 -> lower=-4.77 upper=2.25 effort=150.0 velocity=3.15
- joint wrist_1_joint: limit lower=-6.28318530718 upper=6.28318530718 effort=28.0 velocity=3.2 -> lower=-3.141592653589793 upper=1.5707963267948966 effort=28.0 velocity=3.2; origin xyz=0.0 0.0 0.39225 rpy=0.0 1.57079632679 0.0 -> xyz=0.0 0.0 0.39225 rpy=0.0 1.5707963267948966 0.0
- joint wrist_2_joint: limit lower=-6.28318530718 upper=6.28318530718 effort=28.0 velocity=3.2 -> lower=-1.6 upper=4.74 effort=28.0 velocity=3.2
- joint wrist_3_joint: limit lower=-6.28318530718 upper=6.28318530718 effort=28.0 velocity=3.2 -> lower=0 upper=6.283185307179586 effort=28.0 velocity=3.2
- joint wrist_3_link-tool0_fixed_joint: origin xyz=0 0.0823 0 rpy=-1.57079632679 0 0 -> xyz=0 0.0823 0 rpy=-1.5707963267948966 0 0

Commit message: Moved joint limitation to joint_limites.yaml and changed configuration for planning

File: ur_description/urdf/ur5.urdf.xacro (robot description, xacro)
@@ -101,5 +101,5 @@
       <axis xyz="0 0 1" />
       <xacro:unless value="${joint_limited}">
-        <limit lower="-4.2" upper="2.8" effort="150.0" velocity="3.15"/>
+        <limit lower="${-2.0 * pi}" upper="${2.0 * pi}" effort="150.0" velocity="3.15"/>
         <xacro:if value="${safety_limits}">
           <safety_controller soft_lower_limit="${-2.0 * pi + safety_pos_margin}" soft_upper_limit="${2.0 * pi - safety_pos_margin}" k_position="${safety_k_position}" k_velocity="0.0"/>
@@ -138,5 +138,5 @@
       <axis xyz="0 1 0" />
       <xacro:unless value="${joint_limited}">
-        <limit lower="-3.1" upper="-0.4" effort="150.0" velocity="3.15"/>
+        <limit lower="${-2.0 * pi}" upper="${2.0 * pi}" effort="150.0" velocity="3.15"/>
         <xacro:if value="${safety_limits}">
           <safety_controller soft_lower_limit="${-2.0 * pi + safety_pos_margin}" soft_upper_limit="${2.0 * pi - safety_pos_margin}" k_position="${safety_k_position}" k_velocity="0.0"/>
@@ -175,5 +175,5 @@
       <axis xyz="0 1 0" />
       <xacro:unless value="${joint_limited}">
-        <limit lower="0.6" upper="2.75" effort="150.0" velocity="3.15"/>
+        <limit lower="${-2.0 * pi}" upper="${2.0 * pi}" effort="150.0" velocity="3.15"/>
         <xacro:if value="${safety_limits}">
           <safety_controller soft_lower_limit="${-2.0 * pi + safety_pos_margin}" soft_upper_limit="${2.0 * pi - safety_pos_margin}" k_position="${safety_k_position}" k_velocity="0.0"/>
@@ -212,5 +212,5 @@
       <axis xyz="0 1 0" />
       <xacro:unless value="${joint_limited}">
-        <limit lower="-1.4" upper="1.1" effort="28.0" velocity="3.2"/>
+        <limit lower="${-2.0 * pi}" upper="${2.0 * pi}" effort="28.0" velocity="3.2"/>
         <xacro:if value="${safety_limits}">
           <safety_controller soft_lower_limit="${-2.0 * pi + safety_pos_margin}" soft_upper_limit="${2.0 * pi - safety_pos_margin}" k_position="${safety_k_position}" k_velocity="0.0"/>
@@ -249,5 +249,5 @@
       <axis xyz="0 0 1" />
       <xacro:unless value="${joint_limited}">
-        <limit lower="-1.7" upper="3.0" effort="28.0" velocity="3.2"/>
+        <limit lower="${-2.0 * pi}" upper="${2.0 * pi}" effort="28.0" velocity="3.2"/>
         <xacro:if value="${safety_limits}">
           <safety_controller soft_lower_limit="${-2.0 * pi + safety_pos_margin}" soft_upper_limit="${2.0 * pi - safety_pos_margin}" k_position="${safety_k_position}" k_velocity="0.0"/>
@@ -286,5 +286,5 @@
       <axis xyz="0 1 0" />
       <xacro:unless value="${joint_limited}">
-        <limit lower="-0.35" upper="4.8" effort="28.0" velocity="3.2"/>
+        <limit lower="${-2.0 * pi}" upper="${2.0 * pi}" effort="28.0" velocity="3.2"/>
         <xacro:if value="${safety_limits}">
           <safety_controller soft_lower_limit="${-2.0 * pi + safety_pos_margin}" soft_upper_limit="${2.0 * pi - safety_pos_margin}" k_position="${safety_k_position}" k_velocity="0.0"/>

File: ur_description/urdf/ur5_with_eof.urdf (robot description, URDF)
Before this commit: robot ur5_with_eof, 13 links, 12 joints
Joints:
- joint elbow_joint: limit lower=-0.3 upper=2.84 effort=150.0 velocity=3.15 -> lower=-6.28 upper=6.28 effort=150.0 velocity=3.15
- joint shoulder_lift_joint: limit lower=-2.1 upper=0.0 effort=150.0 velocity=3.15 -> lower=-6.28 upper=6.28 effort=150.0 velocity=3.15
- joint shoulder_pan_joint: limit lower=-4.77 upper=2.25 effort=150.0 velocity=3.15 -> lower=-6.28 upper=6.28 effort=150.0 velocity=3.15
- joint wrist_1_joint: limit lower=-3.141592653589793 upper=1.5707963267948966 effort=28.0 velocity=3.2 -> lower=-6.28 upper=6.28 effort=28.0 velocity=3.2
- joint wrist_2_joint: limit lower=-1.6 upper=4.74 effort=28.0 velocity=3.2 -> lower=-6.28 upper=6.28 effort=28.0 velocity=3.2
- joint wrist_3_joint: limit lower=0 upper=6.283185307179586 effort=28.0 velocity=3.2 -> lower=-6.28 upper=6.28 effort=28.0 velocity=3.2
